File: PCB/cyberdeck.kicad_pcb (KiCad board)
At the start: 2 copper layers, 110.7 x 67.3 mm, 38 parts, among them J1 Conn_01x03, J2 Conn_01x06, J4 Conn_01x12, J5 Conn_01x12, J6 Conn_01x06, M1 MountingHole_3.2mm_M3, M2 MountingHole_3.2mm_M3, M3 MountingHole_3.2mm_M3, M4 MountingHole_3.2mm_M3, M5 MountingHole_3.2mm_M3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

Commit message: Right controller tweaks
Parts:
- R_U1: moved to B.Cu
- turned R_U1 to 180 degrees
Routing:
- net J_JH_SW: track 76.9 -> 63.7 mm, vias 2 -> 4
- net Net-(JH1-Y): track 43.3 -> 35.3 mm
- net J_AGND: track 64.9 -> 61.0 mm, vias 3 -> 2
- net J_3.3v: track 56.1 -> 58.9 mm, vias 0 -> 1
- net J_Trigger_ADC: track 49.5 -> 52.0 mm, vias 0 -> 1
Other:
- board size 110.7 x 67.3 mm -> 110.7 x 67.8 mm
